File: PCB/1001kit-pcb.sch (KiCad schematic (older format))
At the start: 7 parts, among them U1 esp-devkit, U2 MC33926-carrier, U3 arduino-mega, U4 stepper-module, U5 polulu-3784-D36V28F7, U6 pi-display-conn, U7 bob-12009

Commit message: Added IO headers from old shield
IOs added to match old shield.
Parts:
- added J? (x58): Conn_01x03, symbol Connector_Generic:Conn_01x03
- added R? (x48): PTC, symbol Device:R
- added U?: stepper-module, stepper-module:stepper-module, symbol stepper-module:stepper-module
Connections:
- net labels added: 3V-Ana, 3V-Digi, 5V-Ana, 5V-Digi, AN0, AN1, AN10, AN11, AN12, AN13, AN14, AN15, AN2, AN3, AN4, AN5, AN6, AN7, AN8, AN9, AN_BANK0, AN_BANK1, AN_BANK2, AN_BANK3, DC-Servo, DIG0, DIG1, DIG10, DIG11, DIG12, DIG13, DIG14, DIG15, DIG16, DIG17, DIG18, DIG19, DIG2, DIG20, DIG21, DIG22, DIG23, DIG3, DIG4, DIG5, DIG6, DIG7, DIG8, DIG9, DIG_BANK0, DIG_BANK1, DIG_BANK2, DIG_BANK3, DIG_BANK4, DIG_BANK5, GNDA
- wire segments 0 -> 282
Other:
- note added: "Analog Input"
- note added: "Digital Input"
- note added: "for PTC. Use PRG18BB221MB1RB. hold current 14mA. trip current 29mA.\nResistance once tripped over 1 k"
- moved on the sheet: U2

Commit message: Added i2c headers
Parts:
- added J? (x12): Conn_01x04, symbol Connector_Generic:Conn_01x04
- added U?: bob-12009, bob12009:bob-12009, symbol bob-12009:bob-12009
Connections:
- net labels added: GNDD, SCL_3V, SCL_5V, SDA_3V, SDA_5V
- wire segments 282 -> 354
Other:
- note added: "I2C Bus Ports"

Commit message: Added H-Bridges
Parts:
- added J? (x3): Conn_01x03, symbol Connector_Generic:Conn_01x03
- added U? (x3): MC33926-carrier, MC33926-Motor-Driver-Carrier:MC33926-Motor-Driver-Carrier, symbol MC33926-Motor-Driver-Carrier:MC33926-carrier
Connections:
- net labels added: GND, MOT-DC, MOT0-Amps, MOT0-Dir, MOT0-En, MOT0-Pwm, MOT0-Stat, MOT1-Amps, MOT1-Dir, MOT1-En, MOT1-Pwm, MOT1-Stat, MOT2-Amps, MOT2-Dir, MOT2-En, MOT2-Pwm, MOT2-Stat
- wire segments 354 -> 415
Other:
- note added: "H-Bridge Motor Drivers"
